File: ASUS BTF GPU Mini-ITX Adapter.kicad_pcb (KiCad board)
At the start: 2 copper layers, 38 x 25 mm, 2 parts

Commit message: groundplane hotfix
Routing:
- net SENSE1: track 26.9 -> 69.3 mm
- net SENSE0: track 15.4 -> 14.3 mm
